File: Motor Controller PCB/Motor Controller Main Board/MotorControllerMainBoard.sch (EAGLE design)
At the start: 88 parts, among them T1 TEENSY_3.1_ALL_PINS

Commit message: Revert "Added Header, Worked on Digital Connections"
This reverts commit b0afa353cafffa68415efb6e73d521797ab7b560.
Parts:
- removed J1: (no value), SparkFun-Connectors:M03PTH
- removed J2: (no value), SparkFun-Connectors:M05X2NO_SILK
Connections:
- removed net BUTTON1: J2.10, T1.11/MOSI
- removed net BUTTON2: J2.9, T1.12/MISO
- removed net HALL_SENSOR: J1.3, T1.22/A8/T/PWM
- removed net RX_OUT: J2.6, T1.7/RX3
- removed net SCL0: J2.7, T1.19/A5/T/SCL0
- removed net SDA0: J2.5, T1.18/A4/T/SDA0
- removed net TX_OUT: J2.8, T1.8/TX3
- net 12V_POWER_REGULATED: no longer J2.3
- net 5V_POWER_REGULATED: no longer J1.2, J2.4
- net GND: no longer J1.1, J2.1, J2.2
- net SUPPLY_VOLTAGE: now also T1.18/A4/T/SDA0; no longer T1.21/A7/PWM
Other:
- note removed: "Hall Sensor"
- note removed: "IO Header"
Changed lines of the file:
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@@
 <part name="GND33" library="E-P-008-R1.2" deviceset="GND" device=""/>
 <part name="L2" library="SparkFun (2015_10_14 22_27_04 UTC)" deviceset="INDUCTOR" device="0805" value="42nH"/>
-<part name="J2" library="SparkFun-Connectors" deviceset="M05X2" device="NO_SILK"/>
-<part name="J1" library="SparkFun-Connectors" deviceset="M03" device="PTH"/>
 </parts>
 <sheets>
@@
 <text x="223.52" y="58.42" size="1.778" layer="91" rot="R270">Schottky</text>
 <text x="223.52" y="76.2" size="1.778" layer="91" rot="R270">Schottky</text>
-<text x="33.02" y="144.78" size="1.778" layer="95">IO Header</text>
-<text x="25.4" y="111.76" size="1.778" layer="95">Hall Sensor</text>
 </plain>
 <instances>
@@
 <instance part="GND33" gate="1" x="231.14" y="50.8"/>
 <instance part="L2" gate="G$1" x="208.28" y="144.78" rot="R90"/>
-<instance part="J2" gate="G$1" x="38.1" y="129.54"/>
-<instance part="J1" gate="J$1" x="30.48" y="101.6"/>
 </instances>
 <busses>
@@
 <wire x1="231.14" y1="55.88" x2="231.14" y2="53.34" width="0.1524" layer="91"/>
 </segment>
-<segment>
-<pinref part="J2" gate="G$1" pin="1"/>
-<wire x1="30.48" y1="134.62" x2="27.94" y2="134.62" width="0.1524" layer="91"/>
-<label x="22.86" y="134.62" size="1.778" layer="95"/>
-</segment>
-<segment>
-<pinref part="J2" gate="G$1" pin="2"/>
-<wire x1="45.72" y1="134.62" x2="48.26" y2="134.62" width="0.1524" layer="91"/>
-<label x="48.26" y="134.62" size="1.778" layer="95"/>
-</segment>
-<segment>
-<pinref part="J1" gate="J$1" pin="1"/>
-<wire x1="38.1" y1="99.06" x2="40.64" y2="99.06" width="0.1524" layer="91"/>
-<label x="40.64" y="99.06" size="1.778" layer="95"/>
-</segment>
 </net>
 <net name="5V_POWER_REGULATED" class="0">
@@
 <wire x1="83.82" y1="45.72" x2="83.82" y2="43.18" width="0.1524" layer="91"/>
 <label x="71.12" y="40.64" size="1.778" layer="95"/>
-</segment>
-<segment>
-<pinref part="J2" gate="G$1" pin="4"/>
-<wire x1="45.72" y1="132.08" x2="48.26" y2="132.08" width="0.1524" layer="91"/>
-<label x="48.26" y="132.08" size="1.778" layer="95"/>
-</segment>
-<segment>
-<pinref part="J1" gate="J$1" pin="2"/>
-<wire x1="38.1" y1="101.6" x2="40.64" y2="101.6" width="0.1524" layer="91"/>
-<label x="40.64" y="101.6" size="1.778" layer="95"/>
 </segment>
 </net>
@@
 <pinref part="T1" gate="G$1" pin="20/A6/PWM"/>
 <wire x1="116.84" y1="111.76" x2="114.3" y2="111.76" width="0.1524" layer="91"/>
-<label x="93.98" y="111.76" size="1.778" layer="95"/>
+<label x="96.52" y="111.76" size="1.778" layer="95"/>
 </segment>
 </net>
@@
 </segment>
 <segment>
-<pinref part="T1" gate="G$1" pin="21/A7/PWM"/>
-<wire x1="116.84" y1="109.22" x2="114.3" y2="109.22" width="0.1524" layer="91"/>
-<label x="91.44" y="109.22" size="1.778" layer="95"/>
+<pinref part="T1" gate="G$1" pin="18/A4/T/SDA0"/>
+<wire x1="116.84" y1="116.84" x2="114.3" y2="116.84" width="0.1524" layer="91"/>
+<label x="88.9" y="116.84" size="1.778" layer="95"/>
 </segment>
 </net>
@@
 <wire x1="198.12" y1="73.66" x2="200.66" y2="73.66" width="0.1524" layer="91"/>
 <label x="182.88" y="71.12" size="1.778" layer="95"/>
-</segment>
-<segment>
-<pinref part="J2" gate="G$1" pin="3"/>
-<wire x1="30.48" y1="132.08" x2="27.94" y2="132.08" width="0.1524" layer="91"/>
-<label x="5.08" y="132.08" size="1.778" layer="95"/>
 </segment>
 </net>
@@
 </segment>
 </net>
-<net name="BUTTON2" class="0">
-<segment>
-<pinref part="J2" gate="G$1" pin="9"/>
-<wire x1="30.48" y1="124.46" x2="27.94" y2="124.46" width="0.1524" layer="91"/>
-<label x="17.78" y="124.46" size="1.778" layer="95"/>
-</segment>
-<segment>
-<pinref part="T1" gate="G$1" pin="12/MISO"/>
-<wire x1="116.84" y1="132.08" x2="114.3" y2="132.08" width="0.1524" layer="91"/>
-<label x="101.6" y="132.08" size="1.778" layer="95"/>
-</segment>
-</net>
-<net name="BUTTON1" class="0">
-<segment>
-<pinref part="J2" gate="G$1" pin="10"/>
-<wire x1="45.72" y1="124.46" x2="48.26" y2="124.46" width="0.1524" layer="91"/>
-<label x="48.26" y="124.46" size="1.778" layer="95"/>
-</segment>
-<segment>
-<pinref part="T1" gate="G$1" pin="11/MOSI"/>
-<wire x1="116.84" y1="134.62" x2="114.3" y2="134.62" width="0.1524" layer="91"/>
-<label x="101.6" y="134.62" size="1.778" layer="95"/>
-</segment>
-</net>
-<net name="SDA0" class="0">
-<segment>
-<pinref part="T1" gate="G$1" pin="18/A4/T/SDA0"/>
-<wire x1="116.84" y1="116.84" x2="114.3" y2="116.84" width="0.1524" layer="91"/>
-<label x="99.06" y="116.84" size="1.778" layer="95"/>
-</segment>
-<segment>
-<pinref part="J2" gate="G$1" pin="5"/>
-<wire x1="30.48" y1="129.54" x2="27.94" y2="129.54" width="0.1524" layer="91"/>
-<label x="22.86" y="129.54" size="1.778" layer="95"/>
-</segment>
-</net>
-<net name="SCL0" class="0">
-<segment>
-<pinref part="T1" gate="G$1" pin="19/A5/T/SCL0"/>
-<wire x1="116.84" y1="114.3" x2="114.3" y2="114.3" width="0.1524" layer="91"/>
-<label x="99.06" y="114.3" size="1.778" layer="95"/>
-</segment>
-<segment>
-<pinref part="J2" gate="G$1" pin="7"/>
-<wire x1="30.48" y1="127" x2="27.94" y2="127" width="0.1524" layer="91"/>
-<label x="22.86" y="127" size="1.778" layer="95"/>
-</segment>
-</net>
-<net name="RX_OUT" class="0">
-<segment>
-<pinref part="T1" gate="G$1" pin="7/RX3"/>
-<wire x1="116.84" y1="144.78" x2="114.3" y2="144.78" width="0.1524" layer="91"/>
-<label x="104.14" y="144.78" size="1.778" layer="95"/>
-</segment>
-<segment>
-<pinref part="J2" gate="G$1" pin="6"/>
-<wire x1="45.72" y1="129.54" x2="48.26" y2="129.54" width="0.1524" layer="91"/>
-<label x="48.26" y="129.54" size="1.778" layer="95"/>
-</segment>
-</net>
-<net name="TX_OUT" class="0">
-<segment>
-<pinref part="T1" gate="G$1" pin="8/TX3"/>
-<wire x1="116.84" y1="142.24" x2="114.3" y2="142.24" width="0.1524" layer="91"/>
-<label x="104.14" y="142.24" size="1.778" layer="95"/>
-</segment>
-<segment>
-<pinref part="J2" gate="G$1" pin="8"/>
-<wire x1="45.72" y1="127" x2="48.26" y2="127" width="0.1524" layer="91"/>
-<label x="48.26" y="127" size="1.778" layer="95"/>
-</segment>
-</net>
-<net name="HALL_SENSOR" class="0">
-<segment>
-<pinref part="T1" gate="G$1" pin="22/A8/T/PWM"/>
-<wire x1="116.84" y1="106.68" x2="114.3" y2="106.68" width="0.1524" layer="91"/>
-<label x="91.44" y="106.68" size="1.778" layer="95"/>
-</segment>
-<segment>
-<pinref part="J1" gate="J$1" pin="3"/>
-<wire x1="38.1" y1="104.14" x2="40.64" y2="104.14" width="0.1524" layer="91"/>
-<label x="40.64" y="104.14" size="1.778" layer="95"/>
-</segment>
-</net>
