File: Motor Controller PCB/Motor Controller Main Board/MotorControllerMainBoard.brd (EAGLE design)
At the start: 99 x 100 mm, 94 parts, among them T1 TEENSY_3.1_ALL_PINS

Commit message: DRC tweaks
Routing:
- net N$21: track 0.00 -> 4.11 mm
- net 12V_POWER_REGULATED: track 163.2 -> 161.4 mm
- net MOTOR_OUTPUT_(+): track 384.2 -> 382.8 mm
