File: Motor Controller PCB/Motor Controller Power Board/MotorControllerMainBoard.sch (EAGLE design)
At the start: 45 parts

Commit message: Made changes to 12V regulator
Parts:
- removed U$8: 1N5819, MotorControllerEagleLibrary:1N5819
- added U1: CDBA340L-G, MotorControllerEagleLibrary:CDBA340L-G
- U$7: value 330uH -> 100uH
Connections:
- net GND: now also U1.22; no longer U$8.A
- net N$1: now also U1.11; no longer U$8.K
Other:
- note added: "2.8A Rating"
- moved on the sheet: C5, C6, C7, U$7
Changed lines of the file:
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@@
 <?xml version="1.0" encoding="utf-8"?>
 <!DOCTYPE eagle SYSTEM "eagle.dtd">
-<eagle version="8.4.0">
+<eagle version="8.5.2">
 <drawing>
 <settings>
@@
 <part name="FRAME7" library="E-P-008-R1.2" deviceset="FRAME_A_L" device=""/>
 <part name="U$5" library="MotorControllerEagleLibrary" deviceset="FLYBACK" device=""/>
-<part name="U$7" library="MotorControllerEagleLibrary" deviceset="PA4320" device="" value="330uH"/>
-<part name="U$8" library="MotorControllerEagleLibrary" deviceset="1N5819" device=""/>
+<part name="U$7" library="MotorControllerEagleLibrary" deviceset="PA4320" device="" value="100uH"/>
 <part name="C5" library="MotorControllerEagleLibrary" deviceset="EEUFR1H221B" device=""/>
 <part name="C6" library="MotorControllerEagleLibrary" deviceset="EEUFR1H221B" device=""/>
@@
 <part name="FRAME6" library="E-P-008-R1.2" deviceset="FRAME_A_L" device="" value="Voltage_FeedBack"/>
 <part name="U$10" library="MotorControllerEagleLibrary" deviceset="AMC1200BDWVR" device=""/>
+<part name="U1" library="MotorControllerEagleLibrary" deviceset="CDBA340L-G" device=""/>
 </parts>
 <sheets>
@@
 <plain>
 <text x="200.66" y="27.94" size="3.81" layer="94">POWER SUPPLY</text>
-<text x="182.88" y="116.84" size="6.4516" layer="94">12V Supply</text>
-<text x="68.58" y="111.76" size="1.27" layer="94">220uF Panasonic Caps</text>
+<text x="185.42" y="152.4" size="6.4516" layer="94">12V Supply</text>
+<text x="71.12" y="147.32" size="1.27" layer="94">220uF Panasonic Caps</text>
+<text x="68.58" y="157.48" size="1.778" layer="94" rot="R90">2.8A Rating</text>
 </plain>
 <instances>
 <instance part="FRAME5" gate="G$1" x="0" y="0"/>
 <instance part="FRAME5" gate="G$2" x="172.72" y="0"/>
-<instance part="U$7" gate="PA4320_INDUCTOR" x="68.58" y="129.54" rot="R90"/>
-<instance part="U$8" gate="G$1" x="58.42" y="124.46" rot="R90"/>
-<instance part="C5" gate="A" x="91.44" y="109.22" rot="R270"/>
-<instance part="C6" gate="A" x="106.68" y="109.22" rot="R270"/>
-<instance part="U$6" gate="A" x="78.74" y="142.24"/>
-<instance part="GND16" gate="1" x="58.42" y="111.76"/>
-<instance part="GND17" gate="1" x="106.68" y="83.82"/>
-<instance part="GND20" gate="1" x="137.16" y="139.7" rot="R90"/>
-<instance part="GND23" gate="1" x="76.2" y="134.62"/>
-<instance part="C7" gate="A" x="119.38" y="109.22" rot="R270"/>
+<instance part="U$7" gate="PA4320_INDUCTOR" x="71.12" y="165.1" rot="R90"/>
+<instance part="C5" gate="A" x="93.98" y="144.78" rot="R270"/>
+<instance part="C6" gate="A" x="109.22" y="144.78" rot="R270"/>
+<instance part="U$6" gate="A" x="81.28" y="177.8"/>
+<instance part="GND16" gate="1" x="53.34" y="147.32"/>
+<instance part="GND17" gate="1" x="109.22" y="119.38"/>
+<instance part="GND20" gate="1" x="139.7" y="175.26" rot="R90"/>
+<instance part="GND23" gate="1" x="78.74" y="170.18"/>
+<instance part="C7" gate="A" x="121.92" y="144.78" rot="R270"/>
+<instance part="U1" gate="A" x="53.34" y="165.1" rot="R270"/>
 </instances>
 <busses>
@@
 <net name="GND" class="0">
 <segment>
-<pinref part="U$8" gate="G$1" pin="A"/>
-<wire x1="58.42" y1="121.92" x2="58.42" y2="114.3" width="0.1524" layer="91"/>
-<pinref part="GND16" gate="1" pin="GND"/>
-</segment>
-<segment>
-<wire x1="106.68" y1="99.06" x2="106.68" y2="86.36" width="0.1524" layer="91"/>
+<wire x1="109.22" y1="134.62" x2="109.22" y2="121.92" width="0.1524" layer="91"/>
 <pinref part="GND17" gate="1" pin="GND"/>
 </segment>
@@
 <pinref part="U$6" gate="A" pin="!ON/OFF"/>
 <pinref part="U$6" gate="A" pin="EPAD"/>
-<wire x1="116.84" y1="139.7" x2="134.62" y2="139.7" width="0.1524" layer="91"/>
-<wire x1="116.84" y1="142.24" x2="116.84" y2="139.7" width="0.1524" layer="91"/>
-<junction x="116.84" y="139.7"/>
+<wire x1="119.38" y1="175.26" x2="137.16" y2="175.26" width="0.1524" layer="91"/>
+<wire x1="119.38" y1="177.8" x2="119.38" y2="175.26" width="0.1524" layer="91"/>
+<junction x="119.38" y="175.26"/>
 <pinref part="GND20" gate="1" pin="GND"/>
 </segment>
 <segment>
 <pinref part="U$6" gate="A" pin="GND"/>
-<wire x1="81.28" y1="137.16" x2="76.2" y2="137.16" width="0.1524" layer="91"/>
+<wire x1="83.82" y1="172.72" x2="78.74" y2="172.72" width="0.1524" layer="91"/>
 <pinref part="GND23" gate="1" pin="GND"/>
 </segment>
 <segment>
 <pinref part="C5" gate="A" pin="22"/>
-<wire x1="91.44" y1="101.6" x2="91.44" y2="99.06" width="0.1524" layer="91"/>
-<wire x1="91.44" y1="99.06" x2="106.68" y2="99.06" width="0.1524" layer="91"/>
+<wire x1="93.98" y1="137.16" x2="93.98" y2="134.62" width="0.1524" layer="91"/>
+<wire x1="93.98" y1="134.62" x2="109.22" y2="134.62" width="0.1524" layer="91"/>
 <pinref part="C7" gate="A" pin="22"/>
-<wire x1="106.68" y1="99.06" x2="119.38" y2="99.06" width="0.1524" layer="91"/>
-<wire x1="119.38" y1="99.06" x2="119.38" y2="101.6" width="0.1524" layer="91"/>
+<wire x1="109.22" y1="134.62" x2="121.92" y2="134.62" width="0.1524" layer="91"/>
+<wire x1="121.92" y1="134.62" x2="121.92" y2="137.16" width="0.1524" layer="91"/>
 <pinref part="C6" gate="A" pin="22"/>
-<wire x1="106.68" y1="101.6" x2="106.68" y2="99.06" width="0.1524" layer="91"/>
-<junction x="106.68" y="99.06"/>
+<wire x1="109.22" y1="137.16" x2="109.22" y2="134.62" width="0.1524" layer="91"/>
+<junction x="109.22" y="134.62"/>
+</segment>
+<segment>
+<pinref part="U1" gate="A" pin="22"/>
+<pinref part="GND16" gate="1" pin="GND"/>
+<wire x1="53.34" y1="154.94" x2="53.34" y2="149.86" width="0.1524" layer="91"/>
 </segment>
 </net>
 <net name="12V_POWER_REGULATED" class="0">
 <segment>
-<wire x1="91.44" y1="119.38" x2="106.68" y2="119.38" width="0.1524" layer="91"/>
-<wire x1="106.68" y1="119.38" x2="119.38" y2="119.38" width="0.1524" layer="91"/>
+<wire x1="93.98" y1="154.94" x2="109.22" y2="154.94" width="0.1524" layer="91"/>
+<wire x1="109.22" y1="154.94" x2="121.92" y2="154.94" width="0.1524" layer="91"/>
 <pinref part="C6" gate="A" pin="11"/>
-<wire x1="119.38" y1="119.38" x2="137.16" y2="119.38" width="0.1524" layer="91"/>
-<wire x1="106.68" y1="109.22" x2="106.68" y2="119.38" width="0.1524" layer="91"/>
-<junction x="106.68" y="119.38"/>
+<wire x1="121.92" y1="154.94" x2="139.7" y2="154.94" width="0.1524" layer="91"/>
+<wire x1="109.22" y1="144.78" x2="109.22" y2="154.94" width="0.1524" layer="91"/>
+<junction x="109.22" y="154.94"/>
 <pinref part="C5" gate="A" pin="11"/>
-<wire x1="91.44" y1="109.22" x2="91.44" y2="119.38" width="0.1524" layer="91"/>
+<wire x1="93.98" y1="144.78" x2="93.98" y2="154.94" width="0.1524" layer="91"/>
 <pinref part="U$7" gate="PA4320_INDUCTOR" pin="-"/>
-<wire x1="68.58" y1="121.92" x2="68.58" y2="119.38" width="0.1524" layer="91"/>
-<wire x1="68.58" y1="119.38" x2="91.44" y2="119.38" width="0.1524" layer="91"/>
-<junction x="91.44" y="119.38"/>
-<wire x1="137.16" y1="137.16" x2="137.16" y2="119.38" width="0.1524" layer="91"/>
-<junction x="137.16" y="119.38"/>
-<wire x1="137.16" y1="119.38" x2="147.32" y2="119.38" width="0.1524" layer="91"/>
-<label x="144.78" y="119.38" size="1.778" layer="95"/>
+<wire x1="71.12" y1="157.48" x2="71.12" y2="154.94" width="0.1524" layer="91"/>
+<wire x1="71.12" y1="154.94" x2="93.98" y2="154.94" width="0.1524" layer="91"/>
+<junction x="93.98" y="154.94"/>
+<wire x1="139.7" y1="172.72" x2="139.7" y2="154.94" width="0.1524" layer="91"/>
+<junction x="139.7" y="154.94"/>
+<wire x1="139.7" y1="154.94" x2="149.86" y2="154.94" width="0.1524" layer="91"/>
+<label x="147.32" y="154.94" size="1.778" layer="95"/>
 <pinref part="U$6" gate="A" pin="FEEDBACK"/>
-<wire x1="116.84" y1="137.16" x2="137.16" y2="137.16" width="0.1524" layer="91"/>
+<wire x1="119.38" y1="172.72" x2="139.7" y2="172.72" width="0.1524" layer="91"/>
 <pinref part="C7" gate="A" pin="11"/>
-<wire x1="119.38" y1="109.22" x2="119.38" y2="119.38" width="0.1524" layer="91"/>
-<junction x="119.38" y="119.38"/>
+<wire x1="121.92" y1="144.78" x2="121.92" y2="154.94" width="0.1524" layer="91"/>
+<junction x="121.92" y="154.94"/>
 </segment>
 </net>
@@
 <segment>
 <pinref part="U$7" gate="PA4320_INDUCTOR" pin="+"/>
-<wire x1="68.58" y1="137.16" x2="68.58" y2="139.7" width="0.1524" layer="91"/>
+<wire x1="71.12" y1="172.72" x2="71.12" y2="175.26" width="0.1524" layer="91"/>
 <pinref part="U$6" gate="A" pin="OUTPUT"/>
-<wire x1="68.58" y1="139.7" x2="81.28" y2="139.7" width="0.1524" layer="91"/>
-<pinref part="U$8" gate="G$1" pin="K"/>
-<wire x1="58.42" y1="127" x2="58.42" y2="139.7" width="0.1524" layer="91"/>
-<wire x1="68.58" y1="139.7" x2="58.42" y2="139.7" width="0.1524" layer="91"/>
-<junction x="68.58" y="139.7"/>
+<wire x1="71.12" y1="175.26" x2="83.82" y2="175.26" width="0.1524" layer="91"/>
+<wire x1="53.34" y1="165.1" x2="53.34" y2="175.26" width="0.1524" layer="91"/>
+<junction x="71.12" y="175.26"/>
+<wire x1="71.12" y1="175.26" x2="53.34" y2="175.26" width="0.1524" layer="91"/>
+<pinref part="U1" gate="A" pin="11"/>
 </segment>
 </net>
@@
 <segment>
 <pinref part="U$6" gate="A" pin="VIN"/>
-<wire x1="81.28" y1="142.24" x2="73.66" y2="142.24" width="0.1524" layer="91"/>
-<label x="53.34" y="147.32" size="1.778" layer="95"/>
-<wire x1="73.66" y1="142.24" x2="73.66" y2="144.78" width="0.1524" layer="91"/>
+<wire x1="83.82" y1="177.8" x2="76.2" y2="177.8" width="0.1524" layer="91"/>
+<label x="55.88" y="182.88" size="1.778" layer="95"/>
+<wire x1="76.2" y1="177.8" x2="76.2" y2="180.34" width="0.1524" layer="91"/>
 </segment>
 </net>
@@
 packages will not be understood (or retained) with this version.
 </note>
+<note version="8.4" severity="warning">
+Since Version 8.4, EAGLE supports properties for SPICE simulation.
+Probes in schematics and SPICE mapping objects found in parts and library devices
+will not be understood with this version. Update EAGLE to the latest version
+for full support of SPICE simulation.
+</note>
 </compatibility>

Commit message: added some leds, removed voltage fb
Parts:
- removed C24, C27, C28, C29, C30: EEU-FR1H331L, MotorControllerEagleLibrary:EEU-FR1H331L
- added C8: EEUFR1H221B, MotorControllerEagleLibrary:EEUFR1H221B
- added LED1: (no value), led:LEDCHIPLED_1206
- added LED2, LED3: (no value), SparkFun (2015_10_14 22_27_04 UTC):LED1206
- added U$11, U$21, U$8: (no value), MotorControllerEagleLibrary:AL5809-20S1-7
- added U$13, U$18, U$19, U$20: EEU-FM1H102B, MotorControllerEagleLibrary:EEU-FM1H102B
- U$10: value AMC1200BDWVR -> EEU-FM1H102B; device MotorControllerEagleLibrary:AMC1200BDWVR -> MotorControllerEagleLibrary:EEU-FM1H102B
Connections:
- new net N$17: LED1.A, U$11.C
- new net N$4: LED3.C, U$21.A
- new net N$9: LED2.A, U$8.C
- net 12V_POWER_REGULATED: now also C5.POSITIVE, C6.POSITIVE, C7.POSITIVE, C8.POSITIVE, U$8.A; no longer C5.11, C6.11, C7.11
- net 3.3V_POWER_REGULATED: now also LED3.A
- net GND: now also C5.NEGATIVE, C6.NEGATIVE, C7.NEGATIVE, C8.NEGATIVE, LED1.C, LED2.C, U$10.NEGATIVE, U$13.NEGATIVE, U$18.NEGATIVE, U$19.NEGATIVE, U$20.NEGATIVE; no longer C19.2, C20.2, C24.22, C26.2, C27.22, C28.22, C29.22, C30.22, C5.22, C6.22, C7.22, U$9.2
- net GND_ISOLATED: now also C19.2, C20.2, C26.2, U$21.C, U$9.2
- net INPUT_POWER(+): now also U$10.POSITIVE, U$11.A, U$13.POSITIVE, U$18.POSITIVE, U$19.POSITIVE, U$20.POSITIVE; no longer C24.11, C27.11, C28.11, C29.11, C30.11
Other:
- note added: "1000uF Electro. Caps 5mF in total Low ESL, Low ESR"
- note removed: "330uF Electro. Caps 1.65mF in total Low ESL, Low ESR"
